File: ROBOCEK_ONGOING/DAY1/DAY1.kicad_sch (KiCad schematic)
At the start: 0 parts

Commit message: DAY1
Parts:
- added D1: LED, LED_THT:LED_D3.0mm, symbol Device:LED
- added J1: Screw_Terminal_01x02, TerminalBlock_Phoenix:TerminalBlock_Phoenix_MKDS-1,5-2_1x02_P5.00mm_Horizontal, symbol Connector:Screw_Terminal_01x02
- added R1: R, Resistor_THT:R_Axial_DIN0204_L3.6mm_D1.6mm_P5.08mm_Horizontal, symbol Device:R
- added SW1: SW_SPST, Button_Switch_THT:SW_DIP_SPSTx01_Slide_9.78x4.72mm_W7.62mm_P2.54mm, symbol Switch:SW_SPST
Connections:
- new net: D1.2 (A), SW1.2 (B)
- new net: R1.2, SW1.1 (A)
- new net +5V: J1.2 (Pin_2), R1.1
- new net GND: D1.1 (K), J1.1 (Pin_1)
