File: ROBOCEK_KICAD_DAY_2/ROBOCEK_KICAD_DAY_2.kicad_sch (KiCad schematic)
At the start: 0 parts

Commit message: Oush
Parts:
- added C1, C3: C_Polarized, Capacitor_SMD:CP_Elec_3x5.3, symbol Device:C_Polarized
- added C2: C, Capacitor_SMD:C_0201_0603Metric, symbol Device:C
- added D1: D, Diode_SMD:D_0603_1608Metric, symbol Device:D
- added D2: SS34, Diode_SMD:D_SMA, symbol Diode:SS34
- added J1, J2, J3, J4: Conn_01x01_Pin, Connector_Wire:SolderWire-0.1sqmm_1x01_D0.4mm_OD1mm, symbol Connector:Conn_01x01_Pin
- added L1: L, Inductor_SMD:L_12x12mm_H8mm, symbol Device:L
- added U1: LM2596S-5, Package_TO_SOT_SMD:TO-263-5_TabPin3, symbol Regulator_Switching:LM2596S-5
Connections:
- new net: C1.1, C2.1, D1.1 (K), U1.1 (VIN)
- new net: D2.1 (K), L1.1, U1.2 (OUT)
- new net +5V: C3.1, J3.1 (Pin_1), L1.2, U1.4 (FB)
- new net Earth: C1.2, C2.2, C3.2, D2.2 (A), J2.1 (Pin_1), J4.1 (Pin_1), U1.3 (GND), U1.5 (~{ON}/OFF)
- new net VCC: D1.2 (A), J1.1 (Pin_1)
