File: ROBOCEK_ONGOING/DAY2/DAY2.kicad_sch (KiCad schematic)
At the start: 0 parts

Commit message: new
Parts:
- added C1, C3: C_Polarized, symbol Device:C_Polarized
- added C2: C, symbol Device:C
- added D1: D, symbol Device:D
- added D2: SS34, Diode_SMD:D_SMA, symbol Diode:SS34
- added J1, J2, J3, J4: Conn_01x01_Pin, symbol Connector:Conn_01x01_Pin
- added L1: L, symbol Device:L
- added U1: LM2596S-5, Package_TO_SOT_SMD:TO-263-5_TabPin3, symbol Regulator_Switching:LM2596S-5
Connections:
- new net: C1.1, C2.1, D1.1 (K), U1.1 (VIN)
- new net: D2.1 (K), L1.1, U1.2 (OUT)
- new net +5V: C3.1, J3.1 (Pin_1), L1.2, U1.4 (FB)
- new net GND: C1.2, C2.2, C3.2, D2.2 (A), J2.1 (Pin_1), J4.1 (Pin_1), U1.3 (GND), U1.5 (~{ON}/OFF)
- new net VCC: D1.2 (A), J1.1 (Pin_1)

Commit message: new
Parts:
- C1, C3: footprint (none) -> Capacitor_SMD:CP_Elec_3x5.3
- C2: footprint (none) -> Capacitor_SMD:C_0201_0603Metric
- D1: footprint (none) -> Diode_SMD:D_0603_1608Metric
- J1, J2, J3, J4: footprint (none) -> Connector_Wire:SolderWire-0.1sqmm_1x01_D0.4mm_OD1mm
- L1: footprint (none) -> Inductor_SMD:L_12x12mm_H4.5mm
Changed lines of the file:
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@@
 			)
 		)
-		(property "Footprint" ""
+		(property "Footprint" "Diode_SMD:D_0603_1608Metric"
 			(at 67.31 66.04 0)
 			(hide yes)
@@
 			)
 		)
-		(property "Footprint" ""
+		(property "Footprint" "Capacitor_SMD:CP_Elec_3x5.3"
 			(at 78.4352 86.36 0)
 			(hide yes)
@@
 			)
 		)
-		(property "Footprint" ""
+		(property "Footprint" "Connector_Wire:SolderWire-0.1sqmm_1x01_D0.4mm_OD1mm"
 			(at 33.02 93.98 0)
 			(hide yes)
@@
 			)
 		)
-		(property "Footprint" ""
+		(property "Footprint" "Capacitor_SMD:C_0201_0603Metric"
 			(at 86.0552 86.36 0)
 			(hide yes)
@@
 			)
 		)
-		(property "Footprint" ""
+		(property "Footprint" "Connector_Wire:SolderWire-0.1sqmm_1x01_D0.4mm_OD1mm"
 			(at 201.93 64.77 0)
 			(hide yes)
@@
 			)
 		)
-		(property "Footprint" ""
+		(property "Footprint" "Connector_Wire:SolderWire-0.1sqmm_1x01_D0.4mm_OD1mm"
 			(at 200.66 85.09 0)
 			(hide yes)
@@
 			)
 		)
-		(property "Footprint" ""
+		(property "Footprint" "Connector_Wire:SolderWire-0.1sqmm_1x01_D0.4mm_OD1mm"
 			(at 33.02 66.04 0)
 			(hide yes)
@@
 			)
 		)
-		(property "Footprint" ""
+		(property "Footprint" "Inductor_SMD:L_12x12mm_H4.5mm"
 			(at 149.86 71.12 0)
 			(hide yes)
@@
 			)
 		)
-		(property "Footprint" ""
+		(property "Footprint" "Capacitor_SMD:CP_Elec_3x5.3"
 			(at 168.6052 88.9 0)
 			(hide yes)
